File: FET_HVR.sch (KiCad schematic (older format))
At the start: 13 parts, among them J1 Conn_01x01_Female, J2 Conn_01x01_Female, J3 Conn_01x01_Female, Q1 Q_NMOS_GDS, U1 LR8N3-G

Commit message: Add files via upload
Parts:
- D1: footprint (none) -> Resistors_THT:R_Axial_DIN0204_L3.6mm_D1.6mm_P7.62mm_Horizontal
- R1, R2, R3: footprint (none) -> Resistors_THT:R_Axial_DIN0309_L9.0mm_D3.2mm_P12.70mm_Horizontal
- RV1: footprint (none) -> Potentiometers:Potentiometer_Alps_RK09Y_Vertical
- U1: footprint Package_TO_SOT_THT:TO-92_Inline -> TO_SOT_Packages_THT:TO-92_Inline_Narrow_Oval
Changed lines of the file:
@@
 F 0 "RV1" H 5631 4746 50  0000 R CNN
 F 1 "100K" H 5631 4655 50  0000 R CNN
-F 2 "" H 5700 4700 50  0001 C CNN
+F 2 "Potentiometers:Potentiometer_Alps_RK09Y_Vertical" H 5700 4700 50  0001 C CNN
 F 3 "~" H 5700 4700 50  0001 C CNN
 	1    5700 4700
@@
 F 0 "D1" H 7200 2616 50  0000 C CNN
 F 1 "10Vzener" H 7200 2525 50  0000 C CNN
-F 2 "" H 7200 2400 50  0001 C CNN
+F 2 "Resistors_THT:R_Axial_DIN0204_L3.6mm_D1.6mm_P7.62mm_Horizontal" H 7200 2400 50  0001 C CNN
 F 3 "~" H 7200 2400 50  0001 C CNN
 	1    7200 2400
@@
 F 0 "U1" V 5196 3230 50  0000 L CNN
 F 1 "LR8N3-G" V 5105 3230 50  0000 L CNN
-F 2 "Package_TO_SOT_THT:TO-92_Inline" H 5150 3150 50  0001 C CNN
+F 2 "TO_SOT_Packages_THT:TO-92_Inline_Narrow_Oval" H 5150 3150 50  0001 C CNN
 F 3 "http://www.supertex.com/pdf/datasheets/LR8.pdf" H 5150 3100 50  0001 C CNN
 	1    5150 3100
@@
 F 0 "R1" H 6070 2896 50  0000 L CNN
 F 1 "2K" H 6070 2805 50  0000 L CNN
-F 2 "" V 5930 2850 50  0001 C CNN
+F 2 "Resistors_THT:R_Axial_DIN0309_L9.0mm_D3.2mm_P12.70mm_Horizontal" V 5930 2850 50  0001 C CNN
 F 3 "~" H 6000 2850 50  0001 C CNN
 	1    6000 2850
@@
 F 0 "R2" H 6070 3796 50  0000 L CNN
 F 1 "390K" H 6070 3705 50  0000 L CNN
-F 2 "" V 5930 3750 50  0001 C CNN
+F 2 "Resistors_THT:R_Axial_DIN0309_L9.0mm_D3.2mm_P12.70mm_Horizontal" V 5930 3750 50  0001 C CNN
 F 3 "~" H 6000 3750 50  0001 C CNN
 	1    6000 3750
@@
 F 0 "R3" H 6070 4246 50  0000 L CNN
 F 1 "47K" H 6070 4155 50  0000 L CNN
-F 2 "" V 5930 4200 50  0001 C CNN
+F 2 "Resistors_THT:R_Axial_DIN0309_L9.0mm_D3.2mm_P12.70mm_Horizontal" V 5930 4200 50  0001 C CNN
 F 3 "~" H 6000 4200 50  0001 C CNN
 	1    6000 4200
